Commit message: Neue Eigenschaften/Kommentare: - Sensor bleibt fixiert. - Die neuen Launch files erlauben mapping was funktioniert.

File: moro_tf/taurob.urdf (robot description, URDF)
Before this commit: robot taurob, 5 links, 4 joints
Links:
- removed link base_link
- removed link right_rod
- added link base_footprint
- added link base_robot; visual box size=0.9 .6 .3
Joints:
- removed joint base_to_right_rod
- removed joint left_rod_to_left_axis
- added joint base_footpring_joint: type fixed, parent odom, child base_robot
- added joint tilt: type continuous, parent left_rod, child left_axis, origin xyz=0 -0.01 0.1, axis 0 -1 0
- joint base_to_left_rod: parent base_link -> base_robot
